File: pcb/pcb_smd/pcb_smd.kicad_pcb (KiCad board)
At the start: 2 copper layers, 53.3 x 43.2 mm, 50 parts, among them J1 USB_B_Micro, J2 AVR-ISP-6, J3 Conn_01x02, SW1 SW_Push, SW2 SW_Push, SW3 SW_Push, U1 ATmega32U4-MU, U2 LTC-4627, U3 MPXV5010, U4 MPXV5010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

Commit message: remove gerbers
Other:
- board size 53.3 x 43.2 mm -> 53.3 x 47 mm
