File: pcb/pcb_smd/pcb_smd.sch (KiCad schematic (older format))
At the start: 50 parts, among them J1 USB_B_Micro, J2 AVR-ISP-6, J3 Conn_01x02, SW1 SW_Push, SW2 SW_Push, SW3 SW_Push, U1 ATmega32U4-MU, U2 LTC-4627, U3 MPXV5010, U4 MPXV5010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

Commit message: switch pogo size
Parts:
- C1, C10, C12, C13, C2, C4, C6, C8, C9: value C -> 1uF
- C11, C5: value C -> .01uF
- C3: value C -> 0.1uF
- L1: value L -> 47nH
- R1: value R -> 10k
- R4: value R -> 2
Other:
- moved on the sheet: C10, C11
Changed lines of the file:
@@
 Connection ~ 8000 2650
 Connection ~ 8250 1750
-Connection ~ 8350 5150
+Connection ~ 8350 5450
 Connection ~ 8500 2050
 Connection ~ 8500 4700
@@
 	8250 4700 8500 4700
 Wire Wire Line
-	8250 4750 8250 4700
-Wire Wire Line
-	8250 5050 8250 5150
-Wire Wire Line
-	8250 5150 8350 5150
-Wire Wire Line
-	8350 5150 8350 5700
-Wire Wire Line
-	8350 5150 8500 5150
+	8250 5050 8250 4700
+Wire Wire Line
+	8250 5350 8250 5450
+Wire Wire Line
+	8250 5450 8350 5450
+Wire Wire Line
+	8350 5450 8350 5700
+Wire Wire Line
+	8350 5450 8500 5450
 Wire Wire Line
 	8500 2050 7750 2050
@@
 	8500 2650 8500 2550
 Wire Wire Line
-	8500 4700 8500 4750
+	8500 4700 8500 5050
 Wire Wire Line
 	8500 4700 8800 4700
 Wire Wire Line
-	8500 5050 8500 5150
+	8500 5350 8500 5450
 Wire Wire Line
 	8650 1900 8000 1900
@@
 P 4100 1450
 F 0 "L1" H 4153 1495 50  0000 L CNN
-F 1 "L" H 4153 1405 50  0000 L CNN
+F 1 "47nH" H 4153 1405 50  0000 L CNN
 F 2 "Inductor_SMD:L_0603_1608Metric" H 4100 1450 50  0001 C CNN
 F 3 "~" H 4100 1450 50  0001 C CNN
@@
 P 3050 2300
 F 0 "R1" H 3120 2345 50  0000 L CNN
-F 1 "R" H 3120 2255 50  0000 L CNN
+F 1 "10k" H 3120 2255 50  0000 L CNN
 F 2 "Resistor_SMD:R_0603_1608Metric" V 2980 2300 50  0001 C CNN
 F 3 "~" H 3050 2300 50  0001 C CNN
@@
 P 3750 1450
 F 0 "R4" H 3820 1495 50  0000 L CNN
-F 1 "R" H 3820 1405 50  0000 L CNN
+F 1 "2" H 3820 1405 50  0000 L CNN
 F 2 "Resistor_SMD:R_0603_1608Metric" V 3680 1450 50  0001 C CNN
 F 3 "~" H 3750 1450 50  0001 C CNN
@@
 P 3250 4050
 F 0 "C1" H 3135 4005 50  0000 R CNN
-F 1 "C" H 3135 4095 50  0000 R CNN
+F 1 "1uF" H 3135 4095 50  0000 R CNN
 F 2 "Capacitor_SMD:C_0603_1608Metric" H 3288 3900 50  0001 C CNN
 F 3 "~" H 3250 4050 50  0001 C CNN
@@
 P 3750 1800
 F 0 "C2" H 3865 1845 50  0000 L CNN
-F 1 "C" H 3865 1755 50  0000 L CNN
+F 1 "1uF" H 3865 1755 50  0000 L CNN
 F 2 "Capacitor_SMD:C_0603_1608Metric" H 3788 1650 50  0001 C CNN
 F 3 "~" H 3750 1800 50  0001 C CNN
@@
 P 4350 1800
 F 0 "C3" H 4465 1845 50  0000 L CNN
-F 1 "C" H 4465 1755 50  0000 L CNN
+F 1 "0.1uF" H 4465 1755 50  0000 L CNN
 F 2 "Capacitor_SMD:C_0603_1608Metric" H 4388 1650 50  0001 C CNN
 F 3 "~" H 4350 1800 50  0001 C CNN
@@
 P 5750 2250
 F 0 "C13" H 5865 2295 50  0000 L CNN
-F 1 "C" H 5865 2205 50  0000 L CNN
+F 1 "1uF" H 5865 2205 50  0000 L CNN
 F 2 "Capacitor_SMD:C_0603_1608Metric" H 5788 2100 50  0001 C CNN
 F 3 "~" H 5750 2250 50  0001 C CNN
@@
 P 5950 5200
 F 0 "C4" H 6000 5300 50  0000 L CNN
-F 1 "C" H 6000 5100 50  0000 L CNN
+F 1 "1uF" H 6000 5100 50  0000 L CNN
 F 2 "Capacitor_SMD:C_0603_1608Metric" H 5988 5050 50  0001 C CNN
 F 3 "~" H 5950 5200 50  0001 C CNN
@@
 P 6250 5200
 F 0 "C5" H 6300 5300 50  0000 L CNN
-F 1 "C" H 6300 5100 50  0000 L CNN
+F 1 ".01uF" H 6300 5100 50  0000 L CNN
 F 2 "Capacitor_SMD:C_0603_1608Metric" H 6288 5050 50  0001 C CNN
 F 3 "~" H 6250 5200 50  0001 C CNN
@@
 P 7600 5400
 F 0 "C6" H 7650 5500 50  0000 L CNN
-F 1 "C" H 7650 5300 50  0000 L CNN
+F 1 "1uF" H 7650 5300 50  0000 L CNN
 F 2 "Capacitor_SMD:C_0603_1608Metric" H 7638 5250 50  0001 C CNN
 F 3 "~" H 7600 5400 50  0001 C CNN
@@
 P 8000 2400
 F 0 "C8" H 8050 2500 50  0000 L CNN
-F 1 "C" H 8050 2300 50  0000 L CNN
+F 1 "1uF" H 8050 2300 50  0000 L CNN
 F 2 "Capacitor_SMD:C_0603_1608Metric" H 8038 2250 50  0001 C CNN
 F 3 "~" H 8000 2400 50  0001 C CNN
@@
 P 8250 2400
 F 0 "C9" H 8300 2500 50  0000 L CNN
-F 1 "C" H 8300 2300 50  0000 L CNN
+F 1 "1uF" H 8300 2300 50  0000 L CNN
 F 2 "Capacitor_SMD:C_0603_1608Metric" H 8288 2250 50  0001 C CNN
 F 3 "~" H 8250 2400 50  0001 C CNN
@@
 L Device:C C10
 U 1 1 5EBEBA48
-P 8250 4900
-F 0 "C10" H 8300 5000 50  0000 L CNN
-F 1 "C" H 8300 4800 50  0000 L CNN
-F 2 "Capacitor_SMD:C_0603_1608Metric" H 8288 4750 50  0001 C CNN
-F 3 "~" H 8250 4900 50  0001 C CNN
-	1    8250 4900
+P 8250 5200
+F 0 "C10" H 8300 5300 50  0000 L CNN
+F 1 "1uF" H 8300 5100 50  0000 L CNN
+F 2 "Capacitor_SMD:C_0603_1608Metric" H 8288 5050 50  0001 C CNN
+F 3 "~" H 8250 5200 50  0001 C CNN
+	1    8250 5200
 	-1   0    0    -1
 $EndComp
@@
 L Device:C C11
 U 1 1 5EBEBA60
-P 8500 4900
-F 0 "C11" H 8550 5000 50  0000 L CNN
-F 1 "C" H 8550 4800 50  0000 L CNN
-F 2 "Capacitor_SMD:C_0603_1608Metric" H 8538 4750 50  0001 C CNN
-F 3 "~" H 8500 4900 50  0001 C CNN
-	1    8500 4900
+P 8500 5200
+F 0 "C11" H 8550 5300 50  0000 L CNN
+F 1 ".01uF" H 8550 5100 50  0000 L CNN
+F 2 "Capacitor_SMD:C_0603_1608Metric" H 8538 5050 50  0001 C CNN
+F 3 "~" H 8500 5200 50  0001 C CNN
+	1    8500 5200
 	-1   0    0    -1
 $EndComp
@@
 P 9850 5400
 F 0 "C12" H 9900 5500 50  0000 L CNN
-F 1 "C" H 9900 5300 50  0000 L CNN
+F 1 "1uF" H 9900 5300 50  0000 L CNN
 F 2 "Capacitor_SMD:C_0603_1608Metric" H 9888 5250 50  0001 C CNN
 F 3 "~" H 9850 5400 50  0001 C CNN

Commit message: finish smd version
Parts:
- removed C10, C12: 1uF, Capacitor_SMD:C_0603_1608Metric, symbol Device:C
- removed C11: .01uF, Capacitor_SMD:C_0603_1608Metric, symbol Device:C
- removed R17: 470, Resistor_SMD:R_0603_1608Metric, symbol Device:R
- removed U4: MPXV5010, common:DIPSOP-8_W550thou, symbol common:MPXV5010
Connections:
- net labels removed: PRESSURE2, VREF
- wire segments 164 -> 159
Other:
- note added: "Button Input and Debouncing"
- note added: "Optional 2.5V Reference"
- note added: "Pressure Transducer and Filtering"
- note added: "Programming Header"
- note added: "UART TX Debug"
- moved on the sheet: BZ1, C1, C13, C2, C3, C4, C5, C6, C7, C8, C9, D1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

Commit message: fix TX pin, fix VBUS
Parts:
- added J4: Conn_01x03, Connector_PinHeader_2.54mm:PinHeader_1x03_P2.54mm_Vertical, symbol Connector_Generic:Conn_01x03
- R2, R3: value R -> 22
- Y1: value Crystal_GND2_Small -> Resonator
Connections:
- wire segments 159 -> 165
Other:
- note added: "Extra"
- moved on the sheet: C13, C4, C5, C6, C7, C8, C9, D3, D4, D5, J2, J3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
