File: pcb/pcb_proto/pcb_proto.sch (KiCad schematic (older format))
At the start: 18 parts, among them J1 Conn_01x02, J3 CONSOLE, SW1 MODE, SW2 UP, SW3 DOWN, U1 ATmega328P-PU, U2 MPXV5010, U3 LTC-4627, Y1 Resonator_Small

Commit message: update through hole board
Parts:
- removed J1: Conn_01x02, Connector_JST:JST_EH_B2B-EH-A_1x02_P2.50mm_Vertical, symbol Connector_Generic:Conn_01x02
- removed SW1: MODE, common:PTS636 SK43 LFS, symbol Switch:SW_MEC_5G
- removed SW2: UP, common:PTS636 SK43 LFS, symbol Switch:SW_MEC_5G
- removed SW3: DOWN, common:PTS636 SK43 LFS, symbol Switch:SW_MEC_5G
- added J1: Barrel_Jack, Connector_BarrelJack:BarrelJack_Wuerth_6941xx301002, symbol Connector:Barrel_Jack
- added SW1, SW2, SW3: SW_Push, common:SW_PUSH_6mm, symbol common:SW_Push
Other:
- moved on the sheet: BZ1
Changed lines of the file:
@@
 Connection ~ 8650 2900
 Wire Wire Line
-	2300 2650 2600 2650
-Wire Wire Line
-	2300 2750 2600 2750
+	2300 2600 2600 2600
+Wire Wire Line
+	2300 2800 2600 2800
 Wire Wire Line
 	2400 3750 2400 3850
@@
 	2400 4750 2400 4850
 Wire Wire Line
-	2600 2250 2600 2650
-Wire Wire Line
-	2600 2750 2600 3150
+	2600 2250 2600 2600
+Wire Wire Line
+	2600 2800 2600 3150
 Wire Wire Line
 	2900 4150 3150 4150
@@
 	4350 3900 4900 3900
 Wire Wire Line
-	4350 4100 5850 4100
-Wire Wire Line
 	4350 4200 5000 4200
 Wire Wire Line
-	4350 4400 4850 4400
+	4350 4300 4850 4300
+Wire Wire Line
+	4350 4400 5850 4400
 Wire Wire Line
 	4350 4500 4800 4500
@@
 	4800 5150 4800 4500
 Wire Wire Line
-	4850 4400 4850 4900
+	4850 4300 4850 4900
 Wire Wire Line
 	4850 4900 5050 4900
@@
 	4900 3850 4900 3900
 Wire Wire Line
-	4900 4300 4350 4300
-Wire Wire Line
-	4900 4650 4900 4300
+	4900 4100 4350 4100
+Wire Wire Line
+	4900 4650 4900 4100
 Wire Wire Line
 	5000 4300 5000 4350
@@
 	5700 5150 5700 5250
 Wire Wire Line
-	5800 4300 5800 4550
-Wire Wire Line
-	5850 4300 5800 4300
+	5800 4600 5800 4850
+Wire Wire Line
+	5850 4600 5800 4600
 Wire Wire Line
 	6400 3800 6650 3800
@@
 Text Label 4600 2700 2    50   ~ 0
 DIG3
+Text Label 4600 2800 2    50   ~ 0
+b
 Text Label 4600 3300 2    50   ~ 0
 DIG:
@@
 L power:GND #PWR0114
 U 1 1 5EB3C207
-P 5800 4550
-F 0 "#PWR0114" H 5800 4300 50  0001 C CNN
-F 1 "GND" H 5805 4377 50  0000 C CNN
-F 2 "" H 5800 4550 50  0001 C CNN
-F 3 "" H 5800 4550 50  0001 C CNN
-	1    5800 4550
+P 5800 4850
+F 0 "#PWR0114" H 5800 4600 50  0001 C CNN
+F 1 "GND" H 5805 4677 50  0000 C CNN
+F 2 "" H 5800 4850 50  0001 C CNN
+F 3 "" H 5800 4850 50  0001 C CNN
+	1    5800 4850
 	1    0    0    -1
 $EndComp
@@
 $EndComp
 $Comp
-L Connector_Generic:Conn_01x02 J1
-U 1 1 5E8CF4CD
-P 2100 2750
-F 0 "J1" H 2019 2427 50  0000 C CNN
-F 1 "Conn_01x02" H 2019 2518 50  0000 C CNN
-F 2 "Connector_JST:JST_EH_B2B-EH-A_1x02_P2.50mm_Vertical" H 2100 2750 50  0001 C CNN
-F 3 "~" H 2100 2750 50  0001 C CNN
-	1    2100 2750
-	-1   0    0    1
-$EndComp
-$Comp
 L Connector_Generic:Conn_01x02 J3
 U 1 1 5EAA881F
@@
 $EndComp
 $Comp
-L Switch:SW_MEC_5G SW1
-U 1 1 5E88D2EA
+L common:SW_Push SW1
+U 1 1 5E939516
 P 5250 4650
-F 0 "SW1" H 5450 4800 50  0000 C CNN
-F 1 "MODE" H 5450 4700 50  0000 C CNN
-F 2 "common:PTS636 SK43 LFS" H 5250 4850 50  0001 C CNN
-F 3 "http://www.apem.com/int/index.php?controller=attachment&id_attachment=488" H 5250 4850 50  0001 C CNN
+F 0 "SW1" H 5250 4934 50  0000 C CNN
+F 1 "SW_Push" H 5250 4843 50  0000 C CNN
+F 2 "common:SW_PUSH_6mm" H 5250 4850 50  0001 C CNN
+F 3 "" H 5250 4850 50  0001 C CNN
 	1    5250 4650
 	1    0    0    -1
 $EndComp
 $Comp
-L Switch:SW_MEC_5G SW2
-U 1 1 5E88D962
+L common:SW_Push SW2
+U 1 1 5E939A25
 P 5250 4900
-F 0 "SW2" H 5450 5050 50  0000 C CNN
-F 1 "UP" H 5450 4950 50  0000 C CNN
-F 2 "common:PTS636 SK43 LFS" H 5250 5100 50  0001 C CNN
-F 3 "http://www.apem.com/int/index.php?controller=attachment&id_attachment=488" H 5250 5100 50  0001 C CNN
+F 0 "SW2" H 5250 5184 50  0000 C CNN
+F 1 "SW_Push" H 5250 5093 50  0000 C CNN
+F 2 "common:SW_PUSH_6mm" H 5250 5100 50  0001 C CNN
+F 3 "" H 5250 5100 50  0001 C CNN
 	1    5250 4900
 	1    0    0    -1
 $EndComp
 $Comp
-L Switch:SW_MEC_5G SW3
-U 1 1 5E88E16C
+L common:SW_Push SW3
+U 1 1 5E93ADFB
 P 5250 5150
-F 0 "SW3" H 5450 5300 50  0000 C CNN
-F 1 "DOWN" H 5450 5200 50  0000 C CNN
-F 2 "common:PTS636 SK43 LFS" H 5250 5350 50  0001 C CNN
-F 3 "http://www.apem.com/int/index.php?controller=attachment&id_attachment=488" H 5250 5350 50  0001 C CNN
+F 0 "SW3" H 5250 5434 50  0000 C CNN
+F 1 "SW_Push" H 5250 5343 50  0000 C CNN
+F 2 "common:SW_PUSH_6mm" H 5250 5350 50  0001 C CNN
+F 3 "" H 5250 5350 50  0001 C CNN
 	1    5250 5150
 	1    0    0    -1
@@
 L Device:Buzzer BZ1
 U 1 1 5EA93D82
-P 5950 4200
-F 0 "BZ1" H 6103 4228 50  0000 L CNN
-F 1 "Piezo" H 6103 4138 50  0000 L CNN
-F 2 "Buzzer_Beeper:Buzzer_TDK_PS1240P02BT_D12.2mm_H6.5mm" V 5925 4300 50  0001 C CNN
-F 3 "~" V 5925 4300 50  0001 C CNN
-	1    5950 4200
+P 5950 4500
+F 0 "BZ1" H 6103 4528 50  0000 L CNN
+F 1 "Piezo" H 6103 4438 50  0000 L CNN
+F 2 "Buzzer_Beeper:Buzzer_TDK_PS1240P02BT_D12.2mm_H6.5mm" V 5925 4600 50  0001 C CNN
+F 3 "~" V 5925 4600 50  0001 C CNN
+	1    5950 4500
 	1    0    0    -1
 $EndComp
@@
 $EndComp
 $Comp
+L Connector:Barrel_Jack J1
+U 1 1 5E90E0FB
+P 2000 2700
+F 0 "J1" H 2057 3023 50  0000 C CNN
+F 1 "Barrel_Jack" H 2057 2932 50  0000 C CNN
+F 2 "Connector_BarrelJack:BarrelJack_Wuerth_6941xx301002" H 2050 2660 50  0001 C CNN
+F 3 "~" H 2050 2660 50  0001 C CNN
+	1    2000 2700
+	1    0    0    -1
+$EndComp
+$Comp

Commit message: remove gerbers
Parts:
- C1: value C -> 1uF
- C2: value C -> 0.1uF
- SW1: value SW_Push -> MODE
- SW2: value SW_Push -> UP
- SW3: value SW_Push -> DOWN
Other:
- note added: "See NXP Appnote AP1646"
- note added: "UART TX"
- moved on the sheet: J1, R2
Changed lines of the file:
@@
 Connection ~ 8650 2900
 Wire Wire Line
-	2300 2600 2600 2600
-Wire Wire Line
-	2300 2800 2600 2800
-Wire Wire Line
 	2400 3750 2400 3850
 Wire Wire Line
 	2400 4750 2400 4850
 Wire Wire Line
-	2600 2250 2600 2600
-Wire Wire Line
-	2600 2800 2600 3150
+	2550 2800 2850 2800
+Wire Wire Line
+	2550 3000 2850 3000
+Wire Wire Line
+	2850 2450 2850 2800
+Wire Wire Line
+	2850 3000 2850 3350
 Wire Wire Line
 	2900 4150 3150 4150
@@
 	4350 3800 4600 3800
 Wire Wire Line
-	4350 3900 4900 3900
+	4350 3900 5050 3900
 Wire Wire Line
 	4350 4200 5000 4200
@@
 	4850 4900 5050 4900
 Wire Wire Line
-	4900 3500 4900 3550
-Wire Wire Line
-	4900 3850 4900 3900
-Wire Wire Line
 	4900 4100 4350 4100
 Wire Wire Line
@@
 	5000 4300 5000 4350
 Wire Wire Line
+	5050 3500 5050 3550
+Wire Wire Line
+	5050 3850 5050 3900
+Wire Wire Line
 	5050 4650 4900 4650
 Wire Wire Line
 	5050 5150 4800 5150
 Wire Wire Line
-	5100 3100 4950 3100
+	5200 3100 4950 3100
 Wire Wire Line
 	5450 4650 5700 4650
@@
 Wire Wire Line
 	9500 3600 9350 3600
+Text Notes 5400 4050 2    50   ~ 0
+UART TX
+Text Notes 9100 2500 2    50   ~ 0
+See NXP Appnote AP1646
 Text Label 3150 4150 2    50   ~ 0
 MISO
@@
 Text Label 4600 4800 2    50   ~ 0
 c
-Text Label 4650 3900 2    50   ~ 0
-RST
 Text Label 4950 2700 2    50   ~ 0
 MOSI
@@
 Text Label 4950 2900 2    50   ~ 0
 SCK
+Text Label 4950 3900 2    50   ~ 0
+RST
 Text Label 6400 3800 2    50   ~ 0
 a
@@
 L power:+5V #PWR0103
 U 1 1 5E8E2040
-P 2600 2250
-F 0 "#PWR0103" H 2600 2100 50  0001 C CNN
-F 1 "+5V" H 2615 2423 50  0000 C CNN
-F 2 "" H 2600 2250 50  0001 C CNN
-F 3 "" H 2600 2250 50  0001 C CNN
-	1    2600 2250
+P 2850 2450
+F 0 "#PWR0103" H 2850 2300 50  0001 C CNN
+F 1 "+5V" H 2865 2623 50  0000 C CNN
+F 2 "" H 2850 2450 50  0001 C CNN
+F 3 "" H 2850 2450 50  0001 C CNN
+	1    2850 2450
 	1    0    0    -1
 $EndComp
@@
 L power:+5V #PWR0116
 U 1 1 5E92C87D
-P 4900 3500
-F 0 "#PWR0116" H 4900 3350 50  0001 C CNN
-F 1 "+5V" H 4915 3673 50  0000 C CNN
-F 2 "" H 4900 3500 50  0001 C CNN
-F 3 "" H 4900 3500 50  0001 C CNN
-	1    4900 3500
+P 5050 3500
+F 0 "#PWR0116" H 5050 3350 50  0001 C CNN
+F 1 "+5V" H 5065 3673 50  0000 C CNN
+F 2 "" H 5050 3500 50  0001 C CNN
+F 3 "" H 5050 3500 50  0001 C CNN
+	1    5050 3500
 	1    0    0    -1
 $EndComp
@@
 L power:GND #PWR0115
 U 1 1 5E8B95CD
-P 2600 3150
-F 0 "#PWR0115" H 2600 2900 50  0001 C CNN
-F 1 "GND" H 2605 2977 50  0000 C CNN
-F 2 "" H 2600 3150 50  0001 C CNN
-F 3 "" H 2600 3150 50  0001 C CNN
-	1    2600 3150
+P 2850 3350
+F 0 "#PWR0115" H 2850 3100 50  0001 C CNN
+F 1 "GND" H 2855 3177 50  0000 C CNN
+F 2 "" H 2850 3350 50  0001 C CNN
+F 3 "" H 2850 3350 50  0001 C CNN
+	1    2850 3350
 	1    0    0    -1
 $EndComp
@@
 L power:GND #PWR0101
 U 1 1 5E8F35C4
-P 5100 3100
-F 0 "#PWR0101" H 5100 2850 50  0001 C CNN
-F 1 "GND" H 5105 2927 50  0000 C CNN
-F 2 "" H 5100 3100 50  0001 C CNN
-F 3 "" H 5100 3100 50  0001 C CNN
-	1    5100 3100
+P 5200 3100
+F 0 "#PWR0101" H 5200 2850 50  0001 C CNN
+F 1 "GND" H 5205 2927 50  0000 C CNN
+F 2 "" H 5200 3100 50  0001 C CNN
+F 3 "" H 5200 3100 50  0001 C CNN
+	1    5200 3100
 	1    0    0    -1
 $EndComp
@@
 L Device:R R2
 U 1 1 5E92B483
-P 4900 3700
-F 0 "R2" H 4970 3745 50  0000 L CNN
-F 1 "10k" H 4970 3655 50  0000 L CNN
-F 2 "Resistor_THT:R_Axial_DIN0207_L6.3mm_D2.5mm_P7.62mm_Horizontal" V 4830 3700 50  0001 C CNN
-F 3 "~" H 4900 3700 50  0001 C CNN
-	1    4900 3700
+P 5050 3700
+F 0 "R2" H 5120 3745 50  0000 L CNN
+F 1 "10k" H 5120 3655 50  0000 L CNN
+F 2 "Resistor_THT:R_Axial_DIN0207_L6.3mm_D2.5mm_P7.62mm_Horizontal" V 4980 3700 50  0001 C CNN
+F 3 "~" H 5050 3700 50  0001 C CNN
+	1    5050 3700
 	1    0    0    -1
 $EndComp
@@
 P 3350 1700
 F 0 "C1" H 3465 1745 50  0000 L CNN
-F 1 "C" H 3465 1655 50  0000 L CNN
+F 1 "1uF" H 3465 1655 50  0000 L CNN
 F 2 "Capacitor_THT:C_Disc_D5.0mm_W2.5mm_P2.50mm" H 3388 1550 50  0001 C CNN
 F 3 "~" H 3350 1700 50  0001 C CNN
@@
 P 4100 1850
 F 0 "C2" H 4215 1895 50  0000 L CNN
-F 1 "C" H 4215 1805 50  0000 L CNN
+F 1 "0.1uF" H 4215 1805 50  0000 L CNN
 F 2 "Capacitor_THT:C_Disc_D5.0mm_W2.5mm_P2.50mm" H 4138 1700 50  0001 C CNN
 F 3 "~" H 4100 1850 50  0001 C CNN
@@
 U 1 1 5E939516
 P 5250 4650
-F 0 "SW1" H 5250 4934 50  0000 C CNN
-F 1 "SW_Push" H 5250 4843 50  0000 C CNN
+F 0 "SW1" H 5500 4700 50  0000 C CNN
+F 1 "MODE" H 5500 4600 50  0000 C CNN
 F 2 "common:SW_PUSH_6mm" H 5250 4850 50  0001 C CNN
 F 3 "" H 5250 4850 50  0001 C CNN
@@
 U 1 1 5E939A25
 P 5250 4900
-F 0 "SW2" H 5250 5184 50  0000 C CNN
-F 1 "SW_Push" H 5250 5093 50  0000 C CNN
+F 0 "SW2" H 5500 4950 50  0000 C CNN
+F 1 "UP" H 5500 4850 50  0000 C CNN
 F 2 "common:SW_PUSH_6mm" H 5250 5100 50  0001 C CNN
 F 3 "" H 5250 5100 50  0001 C CNN
@@
 U 1 1 5E93ADFB
 P 5250 5150
-F 0 "SW3" H 5250 5434 50  0000 C CNN
-F 1 "SW_Push" H 5250 5343 50  0000 C CNN
+F 0 "SW3" H 5500 5200 50  0000 C CNN
+F 1 "DOWN" H 5500 5100 50  0000 C CNN
 F 2 "common:SW_PUSH_6mm" H 5250 5350 50  0001 C CNN
 F 3 "" H 5250 5350 50  0001 C CNN
@@
 L Connector:Barrel_Jack J1
 U 1 1 5E90E0FB
-P 2000 2700
-F 0 "J1" H 2057 3023 50  0000 C CNN
-F 1 "Barrel_Jack" H 2057 2932 50  0000 C CNN
-F 2 "Connector_BarrelJack:BarrelJack_Wuerth_6941xx301002" H 2050 2660 50  0001 C CNN
-F 3 "~" H 2050 2660 50  0001 C CNN
-	1    2000 2700
-	1    0    0    -1
-$EndComp
+P 2250 2900
+F 0 "J1" H 2307 3223 50  0000 C CNN
+F 1 "Barrel_Jack" H 2307 3132 50  0000 C CNN
+F 2 "Connector_BarrelJack:BarrelJack_Wuerth_6941xx301002" H 2300 2860 50  0001 C CNN
+F 3 "~" H 2300 2860 50  0001 C CNN
+	1    2250 2900
+	1    0    0    -1
+$EndComp

Commit message: button order
Parts:
- SW2: value UP -> DOWN
- SW3: value DOWN -> UP
Changed lines of the file:
@@
 P 5250 4900
 F 0 "SW2" H 5500 4950 50  0000 C CNN
-F 1 "UP" H 5500 4850 50  0000 C CNN
+F 1 "DOWN" H 5500 4850 50  0000 C CNN
 F 2 "common:SW_PUSH_6mm" H 5250 5100 50  0001 C CNN
 F 3 "" H 5250 5100 50  0001 C CNN
@@
 P 5250 5150
 F 0 "SW3" H 5500 5200 50  0000 C CNN
-F 1 "DOWN" H 5500 5100 50  0000 C CNN
+F 1 "UP" H 5500 5100 50  0000 C CNN
 F 2 "common:SW_PUSH_6mm" H 5250 5350 50  0001 C CNN
 F 3 "" H 5250 5350 50  0001 C CNN
